Commit message: crane_plus.urdf.xacro内でuse_gazeboフラグを使ってGazebo関連の処理を条件分岐させる+体裁を整える

File: urdf/crane_plus.gazebo.xacro (robot description, xacro)
@@ -24,10 +24,8 @@
             name_link_4
             name_link_hand
-            config_package
-            config_file_path
             ">
     <gazebo>
       <plugin filename="libign_ros2_control-system.so" name="ign_ros2_control::IgnitionROS2ControlPlugin">
-        <parameters>$(find ${config_package})/${config_file_path}</parameters>
+        <parameters>$(find urdf_seminar)/config/crane_plus_controllers.yaml</parameters>
       </plugin>
     </gazebo>

File: urdf/crane_plus.urdf.xacro (robot description, xacro)
@@ -6,9 +6,10 @@
     xmlns:controller="http://playerstage.sourceforge.net/gazebo/xmlschema/#controller"
     xmlns:interface="http://playerstage.sourceforge.net/gazebo/xmlschema/#interface">
+  <xacro:arg name="use_gazebo" default="false" />
   <xacro:include filename="$(find urdf_seminar)/urdf/crane_plus.xacro"/>
-  <xacro:include filename="$(find urdf_seminar)/urdf/crane_plus.gazebo.xacro"/>
-  <xacro:include filename="$(find urdf_seminar)/urdf/crane_plus.gazebo_ros2_control.xacro"/>
-  <xacro:arg name="gz_control_config_package" default="urdf_seminar" />
-  <xacro:arg name="gz_control_config_file_path" default="config/crane_plus_controllers.yaml" />
+  <xacro:if value="$(arg use_gazebo)">
+    <xacro:include filename="$(find urdf_seminar)/urdf/crane_plus.gazebo.xacro"/>
+    <xacro:include filename="$(find urdf_seminar)/urdf/crane_plus.gazebo_ros2_control.xacro"/>
+  </xacro:if>
   <link name="base_link"/>
   <link name="world"/>
@@ -70,29 +71,29 @@
     <origin xyz="0 0 0"/>
   </xacro:crane_plus>
-  <xacro:gazebo_robot_settings
-    name_link_base="${NAME_LINK_BASE}"
-    name_link_1="${NAME_LINK_1}"
-    name_link_2="${NAME_LINK_2}"
-    name_link_3="${NAME_LINK_3}"
-    name_link_4="${NAME_LINK_4}"
-    name_link_hand="${NAME_LINK_HAND}"
-    config_package="$(arg gz_control_config_package)"
-    config_file_path="$(arg gz_control_config_file_path)" />
-  <xacro:crane_plus_gazebo_ros2_control_settings
-    name="crane_plus"
-    name_joint_1="${NAME_JOINT_1}"
-    name_joint_2="${NAME_JOINT_2}"
-    name_joint_3="${NAME_JOINT_3}"
-    name_joint_4="${NAME_JOINT_4}"
-    name_joint_hand="${NAME_JOINT_HAND}"
-    joint_1_lower_limit="${JOINT_1_LOWER_LIMIT}"
-    joint_1_upper_limit="${JOINT_1_UPPER_LIMIT}"
-    joint_2_lower_limit="${JOINT_2_LOWER_LIMIT}"
-    joint_2_upper_limit="${JOINT_2_UPPER_LIMIT}"
-    joint_3_lower_limit="${JOINT_3_LOWER_LIMIT}"
-    joint_3_upper_limit="${JOINT_3_UPPER_LIMIT}"
-    joint_4_lower_limit="${JOINT_4_LOWER_LIMIT}"
-    joint_4_upper_limit="${JOINT_4_UPPER_LIMIT}"
-    joint_hand_lower_limit="${JOINT_HAND_LOWER_LIMIT}"
-    joint_hand_upper_limit="${JOINT_HAND_UPPER_LIMIT}" />
+  <xacro:if value="$(arg use_gazebo)">
+    <xacro:gazebo_robot_settings
+      name_link_base="${NAME_LINK_BASE}"
+      name_link_1="${NAME_LINK_1}"
+      name_link_2="${NAME_LINK_2}"
+      name_link_3="${NAME_LINK_3}"
+      name_link_4="${NAME_LINK_4}"
+      name_link_hand="${NAME_LINK_HAND}" />
+    <xacro:crane_plus_gazebo_ros2_control_settings
+      name="crane_plus"
+      name_joint_1="${NAME_JOINT_1}"
+      name_joint_2="${NAME_JOINT_2}"
+      name_joint_3="${NAME_JOINT_3}"
+      name_joint_4="${NAME_JOINT_4}"
+      name_joint_hand="${NAME_JOINT_HAND}"
+      joint_1_lower_limit="${JOINT_1_LOWER_LIMIT}"
+      joint_1_upper_limit="${JOINT_1_UPPER_LIMIT}"
+      joint_2_lower_limit="${JOINT_2_LOWER_LIMIT}"
+      joint_2_upper_limit="${JOINT_2_UPPER_LIMIT}"
+      joint_3_lower_limit="${JOINT_3_LOWER_LIMIT}"
+      joint_3_upper_limit="${JOINT_3_UPPER_LIMIT}"
+      joint_4_lower_limit="${JOINT_4_LOWER_LIMIT}"
+      joint_4_upper_limit="${JOINT_4_UPPER_LIMIT}"
+      joint_hand_lower_limit="${JOINT_HAND_LOWER_LIMIT}"
+      joint_hand_upper_limit="${JOINT_HAND_UPPER_LIMIT}" />
+  </xacro:if>
 </robot>

File: urdf/crane_plus.xacro (robot description, xacro)
@@ -19,6 +19,4 @@
     <color rgba="0.3 0.3 1.0 1.0"/>
   </material>
-  <xacro:property name="SCALE_MM" value="0.001"/>
-  <xacro:property name="SCALE_CM" value="0.01"/>
   <xacro:property name="MESH_LINK_BASE" value="urdf_seminar/meshes/visual/body_20201013.stl"/>
   <xacro:property name="MESH_LINK_1" value="urdf_seminar/meshes/visual/Link1_20201013.stl"/>
