Commit message: 不要なマテリアルの定義を削除

File: urdf/crane_plus.xacro (robot description, xacro)
@@ -6,16 +6,4 @@
   <material name="white">
     <color rgba="0.95 0.95 0.95 1.0"/>
-  </material>
-  <material name="silver">
-    <color rgba="0.75 0.75 0.75 1.0"/>
-  </material>
-  <material name="red">
-    <color rgba="1.0 0.3 0.3 1.0"/>
-  </material>
-  <material name="green">
-    <color rgba="0.3 1.0 0.3 1.0"/>
-  </material>
-  <material name="blue">
-    <color rgba="0.3 0.3 1.0 1.0"/>
   </material>
   <xacro:property name="MESH_LINK_BASE" value="urdf_seminar/meshes/visual/body_20201013.stl"/>

Commit message: 各STLファイルのパスは一度しか使わないので変数ではなく直書きに変更

File: urdf/crane_plus.xacro (robot description, xacro)
@@ -7,16 +7,4 @@
     <color rgba="0.95 0.95 0.95 1.0"/>
   </material>
-  <xacro:property name="MESH_LINK_BASE" value="urdf_seminar/meshes/visual/body_20201013.stl"/>
-  <xacro:property name="MESH_LINK_1" value="urdf_seminar/meshes/visual/Link1_20201013.stl"/>
-  <xacro:property name="MESH_LINK_2" value="urdf_seminar/meshes/visual/Link2_20201013.stl"/>
-  <xacro:property name="MESH_LINK_3" value="urdf_seminar/meshes/visual/Link3_20201013.stl"/>
-  <xacro:property name="MESH_LINK_4" value="urdf_seminar/meshes/visual/Link4_20201013.stl"/>
-  <xacro:property name="MESH_LINK_HAND" value="urdf_seminar/meshes/visual/Hand_20201013.stl"/>
-  <xacro:property name="MESH_COLLISION_LINK_BASE" value="urdf_seminar/meshes/collision/body_collision_20201013.stl"/>
-  <xacro:property name="MESH_COLLISION_LINK_1" value="urdf_seminar/meshes/collision/Link1_collision_20201013.stl"/>
-  <xacro:property name="MESH_COLLISION_LINK_2" value="urdf_seminar/meshes/collision/Link2_collision_20201013.stl"/>
-  <xacro:property name="MESH_COLLISION_LINK_3" value="urdf_seminar/meshes/collision/Link3_collision_20201013.stl"/>
-  <xacro:property name="MESH_COLLISION_LINK_4" value="urdf_seminar/meshes/collision/Link4_collision_20201013.stl"/>
-  <xacro:property name="MESH_COLLISION_LINK_HAND" value="urdf_seminar/meshes/collision/Hand_collision_20201013.stl"/>
   <xacro:macro name="crane_plus"
       params="parent
@@ -54,5 +42,5 @@
         <origin xyz="0 0 0" rpy="0 0 0"/>
         <geometry>
-          <mesh filename="package://${MESH_LINK_BASE}"
+          <mesh filename="package://urdf_seminar/meshes/visual/body_20201013.stl"
               scale="1 1 1"/>
         </geometry>
@@ -62,5 +50,5 @@
         <origin xyz="0 0 0" rpy="0 0 0"/>
         <geometry>
-          <mesh filename="package://${MESH_COLLISION_LINK_BASE}"
+          <mesh filename="package://urdf_seminar/meshes/collision/body_collision_20201013.stl"
               scale="1 1 1"/>
         </geometry>
@@ -90,5 +78,5 @@
         <origin xyz="0 0 0" rpy="0 0 ${M_PI}"/>
         <geometry>
-          <mesh filename="package://${MESH_LINK_1}"
+          <mesh filename="package://urdf_seminar/meshes/visual/Link1_20201013.stl"
               scale="1 1 1"/>
         </geometry>
@@ -98,5 +86,5 @@
         <origin xyz="0 0 0" rpy="0 0 ${M_PI}"/>
         <geometry>
-          <mesh filename="package://${MESH_COLLISION_LINK_1}"
+          <mesh filename="package://urdf_seminar/meshes/collision/Link1_collision_20201013.stl"
               scale="1 1 1"/>
         </geometry>
@@ -126,13 +114,13 @@
         <origin xyz="0 0 0" rpy="${M_PI/2} 0 0"/>
         <geometry>
-          <mesh filename="package://${MESH_LINK_2}"
-              scale="1 1 1"/>
-        </geometry>
-        <material name="black"/>
-      </visual>
-      <collision>
-        <origin xyz="0 0 0" rpy="${M_PI/2} 0 0"/>
-        <geometry>
-          <mesh filename="package://${MESH_COLLISION_LINK_2}"
+          <mesh filename="package://urdf_seminar/meshes/visual/Link2_20201013.stl"
+              scale="1 1 1"/>
+        </geometry>
+        <material name="black"/>
+      </visual>
+      <collision>
+        <origin xyz="0 0 0" rpy="${M_PI/2} 0 0"/>
+        <geometry>
+          <mesh filename="package://urdf_seminar/meshes/collision/Link2_collision_20201013.stl"
               scale="1 1 1"/>
         </geometry>
@@ -162,13 +150,13 @@
         <origin xyz="0 0 0" rpy="${M_PI/2} 0 0"/>
         <geometry>
-          <mesh filename="package://${MESH_LINK_3}"
-              scale="1 1 1"/>
-        </geometry>
-        <material name="white"/>
-      </visual>
-      <collision>
-        <origin xyz="0 0 0" rpy="${M_PI/2} 0 0"/>
-        <geometry>
-          <mesh filename="package://${MESH_COLLISION_LINK_3}"
+          <mesh filename="package://urdf_seminar/meshes/visual/Link3_20201013.stl"
+              scale="1 1 1"/>
+        </geometry>
+        <material name="white"/>
+      </visual>
+      <collision>
+        <origin xyz="0 0 0" rpy="${M_PI/2} 0 0"/>
+        <geometry>
+          <mesh filename="package://urdf_seminar/meshes/collision/Link3_collision_20201013.stl"
               scale="1 1 1"/>
         </geometry>
@@ -198,13 +186,13 @@
         <origin xyz="0 0 0" rpy="${M_PI/2} 0 0"/>
         <geometry>
-          <mesh filename="package://${MESH_LINK_4}"
-              scale="1 1 1"/>
-        </geometry>
-        <material name="black"/>
-      </visual>
-      <collision>
-        <origin xyz="0 0 0" rpy="${M_PI/2} 0 0"/>
-        <geometry>
-          <mesh filename="package://${MESH_COLLISION_LINK_4}"
+          <mesh filename="package://urdf_seminar/meshes/visual/Link4_20201013.stl"
+              scale="1 1 1"/>
+        </geometry>
+        <material name="black"/>
+      </visual>
+      <collision>
+        <origin xyz="0 0 0" rpy="${M_PI/2} 0 0"/>
+        <geometry>
+          <mesh filename="package://urdf_seminar/meshes/collision/Link4_collision_20201013.stl"
               scale="1 1 1"/>
         </geometry>
@@ -234,5 +222,5 @@
         <origin xyz="0 0 0" rpy="0 -${M_PI/2} 0"/>
         <geometry>
-          <mesh filename="package://${MESH_LINK_HAND}"
+          <mesh filename="package://urdf_seminar/meshes/visual/Hand_20201013.stl"
               scale="1 1 1"/>
         </geometry>
@@ -242,5 +230,5 @@
         <origin xyz="0 0 0" rpy="0 -${M_PI/2} 0"/>
         <geometry>
-          <mesh filename="package://${MESH_COLLISION_LINK_HAND}"
+          <mesh filename="package://urdf_seminar/meshes/collision/Hand_collision_20201013.stl"
               scale="1 1 1"/>
         </geometry>

Commit message: 慣性モーメントを修正

File: urdf/crane_plus.xacro (robot description, xacro)
@@ -57,7 +57,7 @@
       </collision>
       <inertial>
-        <mass value="0.06645"/>
-        <origin xyz="-1.31E-02 7.00E-06 2.12E-02" rpy="0 ${M_PI/8} 0"/>
-        <inertia ixx="1.66E-05" ixy="1.80E-09" ixz="-5.75E-07" iyy="2.36E-05" iyz="-3.23E-08" izz="1.77E-05"/>
+        <mass value="6.39E-02"/>
+        <origin xyz="-1.30E-02 2.60E-05 2.20E-02" rpy="0 0 0"/>
+        <inertia ixx="1.76E-05" ixy="1.33E-08" ixz="-4.74E-07" iyy="2.22E-05" iyz="-7.85E-09" izz="1.94E-05"/>
       </inertial>
     </link>
@@ -77,5 +77,5 @@
     <link name="${name_link_1}">
       <visual>
-        <origin xyz="0 0 0" rpy="0 0 ${M_PI}"/>
+        <origin xyz="0 0 0" rpy="0 0 0"/>
         <geometry>
           <mesh filename="package://urdf_seminar/meshes/visual/Link1_20201013.stl"
@@ -85,5 +85,5 @@
       </visual>
       <collision>
-        <origin xyz="0 0 0" rpy="0 0 ${M_PI}"/>
+        <origin xyz="0 0 0" rpy="0 0 0"/>
         <geometry>
           <mesh filename="package://urdf_seminar/meshes/collision/Link1_collision_20201013.stl"
@@ -93,7 +93,7 @@
       </collision>
       <inertial>
-        <mass value="0.007729"/>
-        <origin xyz="2.00E-06 0.0 1.09E-02" rpy="0 0 0"/>
-        <inertia ixx="3.43E-06" ixy="0.0" ixz="1.66E-10" iyy="1.30E-06" iyz="0.0" izz="3.05E-06"/>
+        <mass value="8.10E-03"/>
+        <origin xyz="2.00E-06 9.96E-04 1.44E-02" rpy="0 0 0"/>
+        <inertia ixx="3.68E-06" ixy="1.80E-11" ixz="1.79E-10" iyy="1.39E-06" iyz="-1.16E-07" izz="3.22E-06"/>
       </inertial>
     </link>
@@ -129,7 +129,7 @@
       </collision>
       <inertial>
-        <mass value="0.116745"/>
-        <origin xyz="7.99E-04 1.00E-06 4.15E-02" rpy="${M_PI/2} 0 0"/>
-        <inertia ixx="1.25E-04" ixy="6.83E-08" ixz="9.50E-11" iyy="1.92E-05" iyz="0.0" izz="1.19E-04"/>
+        <mass value="1.16E-01"/>
+        <origin xyz="1.00E-06 1.07E-03 4.15E-02" rpy="${M_PI/2} 0 0"/>
+        <inertia ixx="1.23E-04" ixy="6.83E-08" ixz="1.12E-10" iyy="1.88E-05" iyz="0.0" izz="1.17E-04"/>
       </inertial>
     </link>
@@ -165,7 +165,7 @@
       </collision>
       <inertial>
-        <mass value="0.072317"/>
-        <origin xyz="6.45E-04 -1.38E-04 7.01E-02" rpy="${M_PI/2} 0 0"/>
-        <inertia ixx="5.41E-05" ixy="-2.28E-07" ixz="-2.67E-09" iyy="1.60E-05" iyz="-5.35E-07" izz="4.69E-05"/>
+        <mass value="7.23E-02"/>
+        <origin xyz="-1.38E-04 6.46E-04 6.96E-02" rpy="${M_PI/2} 0 0"/>
+        <inertia ixx="5.57E-05" ixy="-2.23E-07" ixz="-2.71E-09" iyy="1.60E-05" iyz="-1.31E-06" izz="4.85E-05"/>
       </inertial>
     </link>
@@ -201,7 +201,7 @@
       </collision>
       <inertial>
-        <mass value="0.08185"/>
-        <origin xyz="6.45E-04 -5.70E-04 4.62E-02" rpy="${M_PI/2} 0 0"/>
-        <inertia ixx="5.91E-05" ixy="-5.11E-08" ixz="3.49E-07" iyy="3.62E-05" iyz="1.37E-05" izz="3.98E-05"/>
+        <mass value="8.19E-02"/>
+        <origin xyz="6.68E-04 1.96E-02 4.60E-02" rpy="${M_PI/2} -${M_PI/2} 0"/>
+        <inertia ixx="3.60E-05" ixy="4.94E-08" ixz="1.34E-05" iyy="6.00E-05" iyz="-5.15E-07" izz="4.04E-05"/>
       </inertial>
     </link>
@@ -237,7 +237,7 @@
       </collision>
       <inertial>
-        <mass value="0.022901"/>
-        <origin xyz="0.0 -2.04E-02 2.77E-02" rpy="0 ${M_PI/2} 0"/>
-        <inertia ixx="5.76E-06" ixy="-4.66E-07" ixz="0.0" iyy="2.76E-05" iyz="0.0" izz="2.52E-05"/>
+        <mass value="2.33E-02"/>
+        <origin xyz="4.77E-04 -2.01E-02 2.73E-02" rpy="0 -${M_PI/2} 0"/>
+        <inertia ixx="6.09E-06" ixy="2.38E-07" ixz="2.20E-07" iyy="2.80E-05" iyz="1.62E-07" izz="2.57E-05"/>
       </inertial>
     </link>

Commit message: 重心姿勢の回転に合わせて重心位置のプラスマイナスを修正

File: urdf/crane_plus.xacro (robot description, xacro)
@@ -130,5 +130,5 @@
       <inertial>
         <mass value="1.16E-01"/>
-        <origin xyz="1.00E-06 1.07E-03 4.15E-02" rpy="${M_PI/2} 0 0"/>
+        <origin xyz="1.00E-06 -1.07E-03 4.15E-02" rpy="${M_PI/2} 0 0"/>
         <inertia ixx="1.23E-04" ixy="6.83E-08" ixz="1.12E-10" iyy="1.88E-05" iyz="0.0" izz="1.17E-04"/>
       </inertial>
@@ -166,5 +166,5 @@
       <inertial>
         <mass value="7.23E-02"/>
-        <origin xyz="-1.38E-04 6.46E-04 6.96E-02" rpy="${M_PI/2} 0 0"/>
+        <origin xyz="-1.38E-04 -6.46E-04 6.96E-02" rpy="${M_PI/2} 0 0"/>
         <inertia ixx="5.57E-05" ixy="-2.23E-07" ixz="-2.71E-09" iyy="1.60E-05" iyz="-1.31E-06" izz="4.85E-05"/>
       </inertial>
@@ -238,5 +238,5 @@
       <inertial>
         <mass value="2.33E-02"/>
-        <origin xyz="4.77E-04 -2.01E-02 2.73E-02" rpy="0 -${M_PI/2} 0"/>
+        <origin xyz="-4.77E-04 -2.01E-02 2.73E-02" rpy="0 -${M_PI/2} 0"/>
         <inertia ixx="6.09E-06" ixy="2.38E-07" ixz="2.20E-07" iyy="2.80E-05" iyz="1.62E-07" izz="2.57E-05"/>
       </inertial>

Commit message: Revert "重心姿勢の回転に合わせて重心位置のプラスマイナスを修正"
This reverts commit a5061a8ebe67cf66e5ab469b4c916f3f0cfe3e06.

File: urdf/crane_plus.xacro (robot description, xacro)
@@ -130,5 +130,5 @@
       <inertial>
         <mass value="1.16E-01"/>
-        <origin xyz="1.00E-06 -1.07E-03 4.15E-02" rpy="${M_PI/2} 0 0"/>
+        <origin xyz="1.00E-06 1.07E-03 4.15E-02" rpy="${M_PI/2} 0 0"/>
         <inertia ixx="1.23E-04" ixy="6.83E-08" ixz="1.12E-10" iyy="1.88E-05" iyz="0.0" izz="1.17E-04"/>
       </inertial>
@@ -166,5 +166,5 @@
       <inertial>
         <mass value="7.23E-02"/>
-        <origin xyz="-1.38E-04 -6.46E-04 6.96E-02" rpy="${M_PI/2} 0 0"/>
+        <origin xyz="-1.38E-04 6.46E-04 6.96E-02" rpy="${M_PI/2} 0 0"/>
         <inertia ixx="5.57E-05" ixy="-2.23E-07" ixz="-2.71E-09" iyy="1.60E-05" iyz="-1.31E-06" izz="4.85E-05"/>
       </inertial>
@@ -238,5 +238,5 @@
       <inertial>
         <mass value="2.33E-02"/>
-        <origin xyz="-4.77E-04 -2.01E-02 2.73E-02" rpy="0 -${M_PI/2} 0"/>
+        <origin xyz="4.77E-04 -2.01E-02 2.73E-02" rpy="0 -${M_PI/2} 0"/>
         <inertia ixx="6.09E-06" ixy="2.38E-07" ixz="2.20E-07" iyy="2.80E-05" iyz="1.62E-07" izz="2.57E-05"/>
       </inertial>

Commit message: Revert "慣性モーメントを修正"
This reverts commit 45cd4229787b61fa65100b14afc81408b84ab949.

File: urdf/crane_plus.xacro (robot description, xacro)
@@ -57,7 +57,7 @@
       </collision>
       <inertial>
-        <mass value="6.39E-02"/>
-        <origin xyz="-1.30E-02 2.60E-05 2.20E-02" rpy="0 0 0"/>
-        <inertia ixx="1.76E-05" ixy="1.33E-08" ixz="-4.74E-07" iyy="2.22E-05" iyz="-7.85E-09" izz="1.94E-05"/>
+        <mass value="0.06645"/>
+        <origin xyz="-1.31E-02 7.00E-06 2.12E-02" rpy="0 ${M_PI/8} 0"/>
+        <inertia ixx="1.66E-05" ixy="1.80E-09" ixz="-5.75E-07" iyy="2.36E-05" iyz="-3.23E-08" izz="1.77E-05"/>
       </inertial>
     </link>
@@ -77,5 +77,5 @@
     <link name="${name_link_1}">
       <visual>
-        <origin xyz="0 0 0" rpy="0 0 0"/>
+        <origin xyz="0 0 0" rpy="0 0 ${M_PI}"/>
         <geometry>
           <mesh filename="package://urdf_seminar/meshes/visual/Link1_20201013.stl"
@@ -85,5 +85,5 @@
       </visual>
       <collision>
-        <origin xyz="0 0 0" rpy="0 0 0"/>
+        <origin xyz="0 0 0" rpy="0 0 ${M_PI}"/>
         <geometry>
           <mesh filename="package://urdf_seminar/meshes/collision/Link1_collision_20201013.stl"
@@ -93,7 +93,7 @@
       </collision>
       <inertial>
-        <mass value="8.10E-03"/>
-        <origin xyz="2.00E-06 9.96E-04 1.44E-02" rpy="0 0 0"/>
-        <inertia ixx="3.68E-06" ixy="1.80E-11" ixz="1.79E-10" iyy="1.39E-06" iyz="-1.16E-07" izz="3.22E-06"/>
+        <mass value="0.007729"/>
+        <origin xyz="2.00E-06 0.0 1.09E-02" rpy="0 0 0"/>
+        <inertia ixx="3.43E-06" ixy="0.0" ixz="1.66E-10" iyy="1.30E-06" iyz="0.0" izz="3.05E-06"/>
       </inertial>
     </link>
@@ -129,7 +129,7 @@
       </collision>
       <inertial>
-        <mass value="1.16E-01"/>
-        <origin xyz="1.00E-06 1.07E-03 4.15E-02" rpy="${M_PI/2} 0 0"/>
-        <inertia ixx="1.23E-04" ixy="6.83E-08" ixz="1.12E-10" iyy="1.88E-05" iyz="0.0" izz="1.17E-04"/>
+        <mass value="0.116745"/>
+        <origin xyz="7.99E-04 1.00E-06 4.15E-02" rpy="${M_PI/2} 0 0"/>
+        <inertia ixx="1.25E-04" ixy="6.83E-08" ixz="9.50E-11" iyy="1.92E-05" iyz="0.0" izz="1.19E-04"/>
       </inertial>
     </link>
@@ -165,7 +165,7 @@
       </collision>
       <inertial>
-        <mass value="7.23E-02"/>
-        <origin xyz="-1.38E-04 6.46E-04 6.96E-02" rpy="${M_PI/2} 0 0"/>
-        <inertia ixx="5.57E-05" ixy="-2.23E-07" ixz="-2.71E-09" iyy="1.60E-05" iyz="-1.31E-06" izz="4.85E-05"/>
+        <mass value="0.072317"/>
+        <origin xyz="6.45E-04 -1.38E-04 7.01E-02" rpy="${M_PI/2} 0 0"/>
+        <inertia ixx="5.41E-05" ixy="-2.28E-07" ixz="-2.67E-09" iyy="1.60E-05" iyz="-5.35E-07" izz="4.69E-05"/>
       </inertial>
     </link>
@@ -201,7 +201,7 @@
       </collision>
       <inertial>
-        <mass value="8.19E-02"/>
-        <origin xyz="6.68E-04 1.96E-02 4.60E-02" rpy="${M_PI/2} -${M_PI/2} 0"/>
-        <inertia ixx="3.60E-05" ixy="4.94E-08" ixz="1.34E-05" iyy="6.00E-05" iyz="-5.15E-07" izz="4.04E-05"/>
+        <mass value="0.08185"/>
+        <origin xyz="6.45E-04 -5.70E-04 4.62E-02" rpy="${M_PI/2} 0 0"/>
+        <inertia ixx="5.91E-05" ixy="-5.11E-08" ixz="3.49E-07" iyy="3.62E-05" iyz="1.37E-05" izz="3.98E-05"/>
       </inertial>
     </link>
@@ -237,7 +237,7 @@
       </collision>
       <inertial>
-        <mass value="2.33E-02"/>
-        <origin xyz="4.77E-04 -2.01E-02 2.73E-02" rpy="0 -${M_PI/2} 0"/>
-        <inertia ixx="6.09E-06" ixy="2.38E-07" ixz="2.20E-07" iyy="2.80E-05" iyz="1.62E-07" izz="2.57E-05"/>
+        <mass value="0.022901"/>
+        <origin xyz="0.0 -2.04E-02 2.77E-02" rpy="0 ${M_PI/2} 0"/>
+        <inertia ixx="5.76E-06" ixy="-4.66E-07" ixz="0.0" iyy="2.76E-05" iyz="0.0" izz="2.52E-05"/>
       </inertial>
     </link>

Commit message: 物理パラメータの修正

File: urdf/crane_plus.xacro (robot description, xacro)
@@ -57,6 +57,6 @@
       </collision>
       <inertial>
-        <mass value="0.06645"/>
-        <origin xyz="-1.31E-02 7.00E-06 2.12E-02" rpy="0 ${M_PI/8} 0"/>
+        <mass value="6.65E-02"/>
+        <origin xyz="-1.31E-02 7.00E-06 2.12E-02" rpy="0 0 0"/>
         <inertia ixx="1.66E-05" ixy="1.80E-09" ixz="-5.75E-07" iyy="2.36E-05" iyz="-3.23E-08" izz="1.77E-05"/>
       </inertial>
@@ -77,5 +77,5 @@
     <link name="${name_link_1}">
       <visual>
-        <origin xyz="0 0 0" rpy="0 0 ${M_PI}"/>
+        <origin xyz="0 0 0" rpy="0 0 0"/>
         <geometry>
           <mesh filename="package://urdf_seminar/meshes/visual/Link1_20201013.stl"
@@ -85,5 +85,5 @@
       </visual>
       <collision>
-        <origin xyz="0 0 0" rpy="0 0 ${M_PI}"/>
+        <origin xyz="0 0 0" rpy="0 0 0"/>
         <geometry>
           <mesh filename="package://urdf_seminar/meshes/collision/Link1_collision_20201013.stl"
@@ -93,5 +93,5 @@
       </collision>
       <inertial>
-        <mass value="0.007729"/>
+        <mass value="7.73E-03"/>
         <origin xyz="2.00E-06 0.0 1.09E-02" rpy="0 0 0"/>
         <inertia ixx="3.43E-06" ixy="0.0" ixz="1.66E-10" iyy="1.30E-06" iyz="0.0" izz="3.05E-06"/>
@@ -129,5 +129,5 @@
       </collision>
       <inertial>
-        <mass value="0.116745"/>
+        <mass value="1.17E-01"/>
         <origin xyz="7.99E-04 1.00E-06 4.15E-02" rpy="${M_PI/2} 0 0"/>
         <inertia ixx="1.25E-04" ixy="6.83E-08" ixz="9.50E-11" iyy="1.92E-05" iyz="0.0" izz="1.19E-04"/>
@@ -165,5 +165,5 @@
       </collision>
       <inertial>
-        <mass value="0.072317"/>
+        <mass value="7.23E-02"/>
         <origin xyz="6.45E-04 -1.38E-04 7.01E-02" rpy="${M_PI/2} 0 0"/>
         <inertia ixx="5.41E-05" ixy="-2.28E-07" ixz="-2.67E-09" iyy="1.60E-05" iyz="-5.35E-07" izz="4.69E-05"/>
@@ -201,5 +201,5 @@
       </collision>
       <inertial>
-        <mass value="0.08185"/>
+        <mass value="8.19E-02"/>
         <origin xyz="6.45E-04 -5.70E-04 4.62E-02" rpy="${M_PI/2} 0 0"/>
         <inertia ixx="5.91E-05" ixy="-5.11E-08" ixz="3.49E-07" iyy="3.62E-05" iyz="1.37E-05" izz="3.98E-05"/>
@@ -237,6 +237,6 @@
       </collision>
       <inertial>
-        <mass value="0.022901"/>
-        <origin xyz="0.0 -2.04E-02 2.77E-02" rpy="0 ${M_PI/2} 0"/>
+        <mass value="2.29E-02"/>
+        <origin xyz="0.0 -2.04E-02 2.77E-02" rpy="0 -${M_PI/2} 0"/>
         <inertia ixx="5.76E-06" ixy="-4.66E-07" ixz="0.0" iyy="2.76E-05" iyz="0.0" izz="2.52E-05"/>
       </inertial>

Commit message: jointのdynamicsをinsert_blockで設定する

File: urdf/crane_plus.xacro (robot description, xacro)
@@ -7,4 +7,7 @@
     <color rgba="0.95 0.95 0.95 1.0"/>
   </material>
+  <xacro:property name="dynamics">
+    <dynamics damping="1.00E-06" friction="0.2"/>
+  </xacro:property>
   <xacro:macro name="crane_plus"
       params="parent
@@ -73,5 +76,5 @@
       <parent link="${name_link_base}"/>
       <child link="${name_link_1}"/>
-      <dynamics damping="1.0e-6" friction="2.0e-1"/>
+      <xacro:insert_block name="dynamics"/>
     </joint>
     <link name="${name_link_1}">
@@ -109,5 +112,5 @@
       <parent link="${name_link_1}"/>
       <child link="${name_link_2}"/>
-      <dynamics damping="1.0e-6" friction="2.0e-1"/>
+      <xacro:insert_block name="dynamics"/>
     </joint>
     <link name="${name_link_2}">
@@ -145,5 +148,5 @@
       <parent link="${name_link_2}"/>
       <child link="${name_link_3}"/>
-      <dynamics damping="1.0e-6" friction="2.0e-1"/>
+      <xacro:insert_block name="dynamics"/>
     </joint>
     <link name="${name_link_3}">
@@ -181,5 +184,5 @@
       <parent link="${name_link_3}"/>
       <child link="${name_link_4}"/>
-      <dynamics damping="1.0e-6" friction="2.0e-1"/>
+      <xacro:insert_block name="dynamics"/>
     </joint>
     <link name="${name_link_4}">
@@ -217,5 +220,5 @@
       <parent link="${name_link_4}"/>
       <child link="${name_link_hand}"/>
-      <dynamics damping="1.0e-6" friction="2.0e-1"/>
+      <xacro:insert_block name="dynamics"/>
     </joint>
     <link name="${name_link_hand}">
