Commit message: meshタグのscaleで改行しない

File: urdf/crane_plus.xacro (robot description, xacro)
@@ -46,14 +46,12 @@
         <origin xyz="0 0 0" rpy="0 0 0"/>
         <geometry>
-          <mesh filename="package://urdf_seminar/meshes/visual/body_20201013.stl"
-              scale="1 1 1"/>
-        </geometry>
-        <material name="black"/>
-      </visual>
-      <collision>
-        <origin xyz="0 0 0" rpy="0 0 0"/>
-        <geometry>
-          <mesh filename="package://urdf_seminar/meshes/collision/body_collision_20201013.stl"
-              scale="1 1 1"/>
+          <mesh filename="package://urdf_seminar/meshes/visual/body_20201013.stl" scale="1 1 1"/>
+        </geometry>
+        <material name="black"/>
+      </visual>
+      <collision>
+        <origin xyz="0 0 0" rpy="0 0 0"/>
+        <geometry>
+          <mesh filename="package://urdf_seminar/meshes/collision/body_collision_20201013.stl" scale="1 1 1"/>
         </geometry>
         <material name="black"/>
@@ -82,14 +80,12 @@
         <origin xyz="0 0 0" rpy="0 0 0"/>
         <geometry>
-          <mesh filename="package://urdf_seminar/meshes/visual/Link1_20201013.stl"
-              scale="1 1 1"/>
-        </geometry>
-        <material name="white"/>
-      </visual>
-      <collision>
-        <origin xyz="0 0 0" rpy="0 0 0"/>
-        <geometry>
-          <mesh filename="package://urdf_seminar/meshes/collision/Link1_collision_20201013.stl"
-              scale="1 1 1"/>
+          <mesh filename="package://urdf_seminar/meshes/visual/Link1_20201013.stl" scale="1 1 1"/>
+        </geometry>
+        <material name="white"/>
+      </visual>
+      <collision>
+        <origin xyz="0 0 0" rpy="0 0 0"/>
+        <geometry>
+          <mesh filename="package://urdf_seminar/meshes/collision/Link1_collision_20201013.stl" scale="1 1 1"/>
         </geometry>
         <material name="white"/>
@@ -118,14 +114,12 @@
         <origin xyz="0 0 0" rpy="${M_PI/2} 0 0"/>
         <geometry>
-          <mesh filename="package://urdf_seminar/meshes/visual/Link2_20201013.stl"
-              scale="1 1 1"/>
-        </geometry>
-        <material name="black"/>
-      </visual>
-      <collision>
-        <origin xyz="0 0 0" rpy="${M_PI/2} 0 0"/>
-        <geometry>
-          <mesh filename="package://urdf_seminar/meshes/collision/Link2_collision_20201013.stl"
-              scale="1 1 1"/>
+          <mesh filename="package://urdf_seminar/meshes/visual/Link2_20201013.stl" scale="1 1 1"/>
+        </geometry>
+        <material name="black"/>
+      </visual>
+      <collision>
+        <origin xyz="0 0 0" rpy="${M_PI/2} 0 0"/>
+        <geometry>
+          <mesh filename="package://urdf_seminar/meshes/collision/Link2_collision_20201013.stl" scale="1 1 1"/>
         </geometry>
         <material name="black"/>
@@ -154,14 +148,12 @@
         <origin xyz="0 0 0" rpy="${M_PI/2} 0 0"/>
         <geometry>
-          <mesh filename="package://urdf_seminar/meshes/visual/Link3_20201013.stl"
-              scale="1 1 1"/>
-        </geometry>
-        <material name="white"/>
-      </visual>
-      <collision>
-        <origin xyz="0 0 0" rpy="${M_PI/2} 0 0"/>
-        <geometry>
-          <mesh filename="package://urdf_seminar/meshes/collision/Link3_collision_20201013.stl"
-              scale="1 1 1"/>
+          <mesh filename="package://urdf_seminar/meshes/visual/Link3_20201013.stl" scale="1 1 1"/>
+        </geometry>
+        <material name="white"/>
+      </visual>
+      <collision>
+        <origin xyz="0 0 0" rpy="${M_PI/2} 0 0"/>
+        <geometry>
+          <mesh filename="package://urdf_seminar/meshes/collision/Link3_collision_20201013.stl" scale="1 1 1"/>
         </geometry>
         <material name="white"/>
@@ -190,14 +182,12 @@
         <origin xyz="0 0 0" rpy="${M_PI/2} 0 0"/>
         <geometry>
-          <mesh filename="package://urdf_seminar/meshes/visual/Link4_20201013.stl"
-              scale="1 1 1"/>
-        </geometry>
-        <material name="black"/>
-      </visual>
-      <collision>
-        <origin xyz="0 0 0" rpy="${M_PI/2} 0 0"/>
-        <geometry>
-          <mesh filename="package://urdf_seminar/meshes/collision/Link4_collision_20201013.stl"
-              scale="1 1 1"/>
+          <mesh filename="package://urdf_seminar/meshes/visual/Link4_20201013.stl" scale="1 1 1"/>
+        </geometry>
+        <material name="black"/>
+      </visual>
+      <collision>
+        <origin xyz="0 0 0" rpy="${M_PI/2} 0 0"/>
+        <geometry>
+          <mesh filename="package://urdf_seminar/meshes/collision/Link4_collision_20201013.stl" scale="1 1 1"/>
         </geometry>
         <material name="black"/>
@@ -226,6 +216,5 @@
         <origin xyz="0 0 0" rpy="0 -${M_PI/2} 0"/>
         <geometry>
-          <mesh filename="package://urdf_seminar/meshes/visual/Hand_20201013.stl"
-              scale="1 1 1"/>
+          <mesh filename="package://urdf_seminar/meshes/visual/Hand_20201013.stl" scale="1 1 1"/>
         </geometry>
         <material name="white"/>
@@ -234,6 +223,5 @@
         <origin xyz="0 0 0" rpy="0 -${M_PI/2} 0"/>
         <geometry>
-          <mesh filename="package://urdf_seminar/meshes/collision/Hand_collision_20201013.stl"
-              scale="1 1 1"/>
+          <mesh filename="package://urdf_seminar/meshes/collision/Hand_collision_20201013.stl" scale="1 1 1"/>
         </geometry>
         <material name="white"/>

Commit message: Revert "jointのdynamicsをinsert_blockで設定する"
This reverts commit 9e5b86a4a9344899d9ede5ddd97eaf8ab7fc5377.

File: urdf/crane_plus.xacro (robot description, xacro)
@@ -7,7 +7,4 @@
     <color rgba="0.95 0.95 0.95 1.0"/>
   </material>
-  <xacro:property name="dynamics">
-    <dynamics damping="1.00E-06" friction="0.2"/>
-  </xacro:property>
   <xacro:macro name="crane_plus"
       params="parent
@@ -74,5 +71,5 @@
       <parent link="${name_link_base}"/>
       <child link="${name_link_1}"/>
-      <xacro:insert_block name="dynamics"/>
+      <dynamics damping="1.0e-6" friction="2.0e-1"/>
     </joint>
     <link name="${name_link_1}">
@@ -108,5 +105,5 @@
       <parent link="${name_link_1}"/>
       <child link="${name_link_2}"/>
-      <xacro:insert_block name="dynamics"/>
+      <dynamics damping="1.0e-6" friction="2.0e-1"/>
     </joint>
     <link name="${name_link_2}">
@@ -142,5 +139,5 @@
       <parent link="${name_link_2}"/>
       <child link="${name_link_3}"/>
-      <xacro:insert_block name="dynamics"/>
+      <dynamics damping="1.0e-6" friction="2.0e-1"/>
     </joint>
     <link name="${name_link_3}">
@@ -176,5 +173,5 @@
       <parent link="${name_link_3}"/>
       <child link="${name_link_4}"/>
-      <xacro:insert_block name="dynamics"/>
+      <dynamics damping="1.0e-6" friction="2.0e-1"/>
     </joint>
     <link name="${name_link_4}">
@@ -210,5 +207,5 @@
       <parent link="${name_link_4}"/>
       <child link="${name_link_hand}"/>
-      <xacro:insert_block name="dynamics"/>
+      <dynamics damping="1.0e-6" friction="2.0e-1"/>
     </joint>
     <link name="${name_link_hand}">

Commit message: dynamicsはinsert_blockではなく直接記述。表記は統一するために修正

File: urdf/crane_plus.xacro (robot description, xacro)
@@ -71,5 +71,5 @@
       <parent link="${name_link_base}"/>
       <child link="${name_link_1}"/>
-      <dynamics damping="1.0e-6" friction="2.0e-1"/>
+      <dynamics damping="1.0E-06" friction="0.2"/>
     </joint>
     <link name="${name_link_1}">
@@ -105,5 +105,5 @@
       <parent link="${name_link_1}"/>
       <child link="${name_link_2}"/>
-      <dynamics damping="1.0e-6" friction="2.0e-1"/>
+      <dynamics damping="1.0E-06" friction="0.2"/>
     </joint>
     <link name="${name_link_2}">
@@ -139,5 +139,5 @@
       <parent link="${name_link_2}"/>
       <child link="${name_link_3}"/>
-      <dynamics damping="1.0e-6" friction="2.0e-1"/>
+      <dynamics damping="1.0E-06" friction="0.2"/>
     </joint>
     <link name="${name_link_3}">
@@ -173,5 +173,5 @@
       <parent link="${name_link_3}"/>
       <child link="${name_link_4}"/>
-      <dynamics damping="1.0e-6" friction="2.0e-1"/>
+      <dynamics damping="1.0E-06" friction="0.2"/>
     </joint>
     <link name="${name_link_4}">
@@ -207,5 +207,5 @@
       <parent link="${name_link_4}"/>
       <child link="${name_link_hand}"/>
-      <dynamics damping="1.0e-6" friction="2.0e-1"/>
+      <dynamics damping="1.0E-06" friction="0.2"/>
     </joint>
     <link name="${name_link_hand}">
